Commit message: fixed collision primitives to cylinders for easier simulations

File: CAD/encoder.urdf (robot description, URDF)
Before this commit: robot encoder, 2 links, 1 joints
Links:
- link rotor: geometry collision cylinder length=17.6 radius=13.45; visual mesh filename=stl/rotor-coarse.STL
- link stator: geometry collision cylinder length=20.88 radius=21; visual mesh filename=stl/stator-coarse.STL
