File: PCB/adapter-encoder-pcb.kicad_sch (KiCad schematic)
At the start: 33 parts, among them IC2 THVD2410VDRCR, M1 THRU_HOLE_PAD, M2 THRU_HOLE_PAD, U1 TLE5009E1000FUMA1, U2 STM32G031G6U6, U3 DF52-4S-0.8H(21), U4 SPX3819M5-L-3-3, U5 C2901617, U6 DF52-4S-0.8H(21), U7 SPX3819M5-L-3-3

Commit message: removed bad biasing resistors
Parts:
- removed R16, R8: 1k, adapter-encoder:R_0402_1005Metric, symbol adapter-encoder:R
Changed lines of the file:
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@@
-    (stroke (width 0) (type default))
-  )
-  (wire (pts (xy 229.87 64.516) (xy 229.87 66.04))
     (stroke (width 0) (type default))
   )
@@
     (stroke (width 0) (type default))
   )
-  (wire (pts (xy 229.87 85.09) (xy 229.87 86.36))
-    (stroke (width 0) (type default))
-  )
   (wire (pts (xy 215.9 83.82) (xy 217.17 83.82))
     (stroke (width 0) (type default))
@@
   )
   (wire (pts (xy 176.53 147.32) (xy 180.975 147.32))
-    (stroke (width 0) (type default))
-  )
-  (wire (pts (xy 229.87 73.66) (xy 229.87 74.93))
     (stroke (width 0) (type default))
   )
@@
   )
   (label "+5V0" (at 193.04 137.16 0) (fields_autoplaced)
-    (effects (font (size 1.27 1.27)) (justify left bottom))
-  )
-  (label "+5V0" (at 229.87 64.516 0) (fields_autoplaced)
     (effects (font (size 1.27 1.27)) (justify left bottom))
   )
@@
     )
   )
-  (symbol (lib_id "power:GND") (at 229.87 93.98 0) (mirror y) (unit 1)
-    (in_bom yes) (on_board yes) (dnp no) (fields_autoplaced)
-    (property "Reference" "#PWR094" (at 229.87 100.33 0)
-      (effects (font (size 1.27 1.27)) hide)
-    )
-    (property "Value" "GND" (at 229.87 99.06 0)
-      (effects (font (size 1.27 1.27)))
-    )
-    (property "Footprint" "" (at 229.87 93.98 0)
-      (effects (font (size 1.27 1.27)) hide)
-    )
-    (property "Datasheet" "" (at 229.87 93.98 0)
-      (effects (font (size 1.27 1.27)) hide)
-    )
-    (pin "1")
-    (instances
-      (project "foc-pcb"
-        (path "/2b52ab19-a93e-4439-8602-a1380e4825c0"
-          (reference "#PWR094") (unit 1)
-        )
-      )
-      (project "adapter-encoder-pcb"
-        (path "/f797ebd5-a509-471a-ba0b-2cd9c6e772fd"
-          (reference "#PWR018") (unit 1)
-        )
-      )
-    )
-  )
   (symbol (lib_id "power:GND") (at 31.75 78.74 0) (unit 1)
     (in_bom yes) (on_board yes) (dnp no) (fields_autoplaced)
@@
     )
   )
-  (symbol (lib_id "adapter-encoder:R") (at 229.87 90.17 0) (mirror x) (unit 1)
-    (in_bom yes) (on_board yes) (dnp no)
-    (property "Reference" "R16" (at 232.41 92.71 0)
-      (effects (font (size 1.27 1.27)) (justify left))
-    )
-    (property "Value" "1k" (at 233.68 90.17 0)
-      (effects (font (size 1.27 1.27)))
-    )
-    (property "Footprint" "adapter-encoder:R_0402_1005Metric" (at 224.79 102.87 0)
-      (effects (font (size 1.27 1.27)) hide)
-    )
-    (property "Datasheet" "~" (at 229.87 90.17 0)
-      (effects (font (size 1.27 1.27)) hide)
-    )
-    (pin "1")
-    (pin "2")
-    (instances
-      (project "foc-pcb"
-        (path "/2b52ab19-a93e-4439-8602-a1380e4825c0"
-          (reference "R16") (unit 1)
-        )
-      )
-      (project "adapter-encoder-pcb"
-        (path "/f797ebd5-a509-471a-ba0b-2cd9c6e772fd"
-          (reference "R4") (unit 1)
-        )
-      )
-    )
-  )
   (symbol (lib_id "power:GND") (at 72.39 110.49 0) (unit 1)
     (in_bom yes) (on_board yes) (dnp no) (fields_autoplaced)
@@
         )
       )
-    )
-  )
-  (symbol (lib_id "adapter-encoder:R") (at 229.87 69.85 0) (mirror x) (unit 1)
-    (in_bom yes) (on_board yes) (dnp no)
-    (property "Reference" "R8" (at 232.41 72.39 0)
-      (effects (font (size 1.27 1.27)) (justify left))
-    )
-    (property "Value" "1k" (at 233.68 69.85 0)
-      (effects (font (size 1.27 1.27)))
-    )
-    (property "Footprint" "adapter-encoder:R_0402_1005Metric" (at 224.79 82.55 0)
-      (effects (font (size 1.27 1.27)) hide)
-    )
-    (property "Datasheet" "~" (at 229.87 69.85 0)
-      (effects (font (size 1.27 1.27)) hide)
-    )
-    (pin "1")
-    (pin "2")
-    (instances
-      (project "foc-pcb"
-        (path "/2b52ab19-a93e-4439-8602-a1380e4825c0"
-          (reference "R8") (unit 1)
-        )
-      )
-      (project "adapter-encoder-pcb"
-        (path "/f797ebd5-a509-471a-ba0b-2cd9c6e772fd"
-          (reference "R2") (unit 1)
-        )
-      )
